File: The Luwu PCB/LED Driver.kicad_sch (KiCad schematic)
At the start: 6 parts, among them IC3 UCC27519DBVR, Q1 BUK7D25-40EX

Commit message: updated README
Parts:
- renumbered C20 to C21, C19 to C22, IC3 to IC6, Q1 to Q2, R4 to R12, R7 to R8
Changed lines of the file:
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@@
   (symbol (lib_id "Device:C") (at 88.265 69.215 0) (unit 1)
     (in_bom yes) (on_board yes) (dnp no) (fields_autoplaced)
-    (property "Reference" "C19" (at 91.44 68.58 0)
+    (property "Reference" "C22" (at 91.44 68.58 0)
       (effects (font (size 1.27 1.27)) (justify left))
     )
@@
   (symbol (lib_id "SamacSys_Parts_2:UCC27519DBVR") (at 106.045 64.135 0) (unit 1)
     (in_bom yes) (on_board yes) (dnp no) (fields_autoplaced)
-    (property "Reference" "IC3" (at 118.745 57.785 0)
+    (property "Reference" "IC6" (at 118.745 57.785 0)
       (effects (font (size 1.27 1.27)))
     )
@@
   (symbol (lib_id "SamacSys_Parts_2:BUK7D25-40EX") (at 143.51 64.135 0) (unit 1)
     (in_bom yes) (on_board yes) (dnp no) (fields_autoplaced)
-    (property "Reference" "Q1" (at 165.735 63.8175 0)
+    (property "Reference" "Q2" (at 165.735 63.8175 0)
       (effects (font (size 1.27 1.27)) (justify left))
     )
@@
   (symbol (lib_id "Device:R") (at 139.065 64.135 90) (unit 1)
     (in_bom yes) (on_board yes) (dnp no)
-    (property "Reference" "R7" (at 139.065 60.325 90)
+    (property "Reference" "R8" (at 139.065 60.325 90)
       (effects (font (size 1.27 1.27)))
     )
@@
   (symbol (lib_id "power:GND") (at 118.745 85.09 0) (unit 1)
     (in_bom yes) (on_board yes) (dnp no) (fields_autoplaced)
-    (property "Reference" "#PWR032" (at 118.745 91.44 0)
+    (property "Reference" "#PWR038" (at 118.745 91.44 0)
       (effects (font (size 1.27 1.27)) hide)
     )
@@
   (symbol (lib_id "Device:R_Small") (at 104.14 67.31 0) (mirror y) (unit 1)
     (in_bom yes) (on_board yes) (dnp no)
-    (property "Reference" "R4" (at 102.235 66.675 0)
+    (property "Reference" "R12" (at 102.235 66.675 0)
       (effects (font (size 1.27 1.27)) (justify left))
     )
@@
   (symbol (lib_id "Device:C") (at 77.47 69.215 0) (unit 1)
     (in_bom yes) (on_board yes) (dnp no) (fields_autoplaced)
-    (property "Reference" "C20" (at 80.645 68.58 0)
-      (effects (font (size 1.27 1.27)) (justify left))
-    )
+    (property "Reference" "C21" (at 80.645 68.58 0)
+      (effects (font (size 1.27 1.27)) (justify left))
+    )
