File: The Luwu PCB/The Luwu PCB.kicad_sch (KiCad schematic)
At the start: 15 parts, among them IC5 SN74LV1T04DCKRG4, J10 Neopixel Terminal out 3, J3 5V_IN, J4 Neopixel Terminal opt 1, J5 12V_IN, J6 V SEL LS, J7 Screw_Terminal_01x04, J8 Neopixel Terminal, J9 Neopixel Terminal opt 2

Commit message: updated README
Parts:
- added H1, H2, H3, H4: MountingHole_Pad, MountingHole:MountingHole_3.2mm_M3_DIN965_Pad, symbol Mechanical:MountingHole_Pad
Connections:
- net GND: now also H1.1, H2.1, H3.1, H4.1
Changed lines of the file:
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@@
+    (stroke (width 0) (type default))
+  )
+  (wire (pts (xy 24.765 146.685) (xy 24.765 149.225))
     (stroke (width 0) (type default))
   )
@@
     (stroke (width 0) (type default))
   )
+  (wire (pts (xy 70.485 146.685) (xy 70.485 149.225))
+    (stroke (width 0) (type default))
+  )
   (wire (pts (xy 217.17 110.49) (xy 195.58 110.49))
     (stroke (width 0) (type default))
@@
   )
   (wire (pts (xy 145.415 19.05) (xy 145.415 59.055))
+    (stroke (width 0) (type default))
+  )
+  (wire (pts (xy 47.625 146.685) (xy 47.625 149.225))
+    (stroke (width 0) (type default))
+  )
+  (wire (pts (xy 93.345 146.685) (xy 93.345 149.225))
     (stroke (width 0) (type default))
   )
@@
   (label "DATA OPT3" (at 151.765 36.83 0) (fields_autoplaced)
     (effects (font (size 1.27 1.27)) (justify left bottom))
+  )
+  (symbol (lib_id "Mechanical:MountingHole_Pad") (at 24.765 144.145 0) (unit 1)
+    (in_bom yes) (on_board yes) (dnp no) (fields_autoplaced)
+    (property "Reference" "H1" (at 27.94 142.24 0)
+      (effects (font (size 1.27 1.27)) (justify left))
+    )
+    (property "Value" "MountingHole_Pad" (at 27.94 144.78 0)
+      (effects (font (size 1.27 1.27)) (justify left))
+    )
+    (property "Footprint" "MountingHole:MountingHole_3.2mm_M3_DIN965_Pad" (at 24.765 144.145 0)
+      (effects (font (size 1.27 1.27)) hide)
+    )
+    (property "Datasheet" "~" (at 24.765 144.145 0)
+      (effects (font (size 1.27 1.27)) hide)
+    )
+    (pin "1")
+    (instances
+      (project "The Luwu PCB"
+        (path "/12a97621-0282-4218-86a3-43268902dd9c"
+          (reference "H1") (unit 1)
+        )
+      )
+    )
   )
   (symbol (lib_id "power:+5V") (at 215.265 34.29 90) (unit 1)
@@
     )
   )
+  (symbol (lib_id "Mechanical:MountingHole_Pad") (at 70.485 144.145 0) (unit 1)
+    (in_bom yes) (on_board yes) (dnp no) (fields_autoplaced)
+    (property "Reference" "H3" (at 73.66 142.24 0)
+      (effects (font (size 1.27 1.27)) (justify left))
+    )
+    (property "Value" "MountingHole_Pad" (at 73.66 144.78 0)
+      (effects (font (size 1.27 1.27)) (justify left))
+    )
+    (property "Footprint" "MountingHole:MountingHole_3.2mm_M3_DIN965_Pad" (at 70.485 144.145 0)
+      (effects (font (size 1.27 1.27)) hide)
+    )
+    (property "Datasheet" "~" (at 70.485 144.145 0)
+      (effects (font (size 1.27 1.27)) hide)
+    )
+    (pin "1")
+    (instances
+      (project "The Luwu PCB"
+        (path "/12a97621-0282-4218-86a3-43268902dd9c"
+          (reference "H3") (unit 1)
+        )
+      )
+    )
+  )
   (symbol (lib_id "power:+12V") (at 131.445 36.83 270) (unit 1)
     (in_bom yes) (on_board yes) (dnp no) (fields_autoplaced)
@@
         (path "/12a97621-0282-4218-86a3-43268902dd9c"
           (reference "#PWR035") (unit 1)
+        )
+      )
+    )
+  )
+  (symbol (lib_id "power:GND") (at 93.345 149.225 0) (unit 1)
+    (in_bom yes) (on_board yes) (dnp no) (fields_autoplaced)
+    (property "Reference" "#PWR052" (at 93.345 155.575 0)
+      (effects (font (size 1.27 1.27)) hide)
+    )
+    (property "Value" "GND" (at 93.345 153.67 0)
+      (effects (font (size 1.27 1.27)))
+    )
+    (property "Footprint" "" (at 93.345 149.225 0)
+      (effects (font (size 1.27 1.27)) hide)
+    )
+    (property "Datasheet" "" (at 93.345 149.225 0)
+      (effects (font (size 1.27 1.27)) hide)
+    )
+    (pin "1")
+    (instances
+      (project "The Luwu PCB"
+        (path "/12a97621-0282-4218-86a3-43268902dd9c"
+          (reference "#PWR052") (unit 1)
         )
       )
@@
     )
   )
+  (symbol (lib_id "Mechanical:MountingHole_Pad") (at 93.345 144.145 0) (unit 1)
+    (in_bom yes) (on_board yes) (dnp no) (fields_autoplaced)
+    (property "Reference" "H4" (at 96.52 142.24 0)
+      (effects (font (size 1.27 1.27)) (justify left))
+    )
+    (property "Value" "MountingHole_Pad" (at 96.52 144.78 0)
+      (effects (font (size 1.27 1.27)) (justify left))
+    )
+    (property "Footprint" "MountingHole:MountingHole_3.2mm_M3_DIN965_Pad" (at 93.345 144.145 0)
+      (effects (font (size 1.27 1.27)) hide)
+    )
+    (property "Datasheet" "~" (at 93.345 144.145 0)
+      (effects (font (size 1.27 1.27)) hide)
+    )
+    (pin "1")
+    (instances
+      (project "The Luwu PCB"
+        (path "/12a97621-0282-4218-86a3-43268902dd9c"
+          (reference "H4") (unit 1)
+        )
+      )
+    )
+  )
   (symbol (lib_id "power:GND") (at 38.735 94.615 0) (unit 1)
     (in_bom yes) (on_board yes) (dnp no) (fields_autoplaced)
@@
     )
   )
+  (symbol (lib_id "Mechanical:MountingHole_Pad") (at 47.625 144.145 0) (unit 1)
+    (in_bom yes) (on_board yes) (dnp no) (fields_autoplaced)
+    (property "Reference" "H2" (at 50.8 142.24 0)
+      (effects (font (size 1.27 1.27)) (justify left))
+    )
+    (property "Value" "MountingHole_Pad" (at 50.8 144.78 0)
+      (effects (font (size 1.27 1.27)) (justify left))
+    )
+    (property "Footprint" "MountingHole:MountingHole_3.2mm_M3_DIN965_Pad" (at 47.625 144.145 0)
+      (effects (font (size 1.27 1.27)) hide)
+    )
+    (property "Datasheet" "~" (at 47.625 144.145 0)
+      (effects (font (size 1.27 1.27)) hide)
+    )
+    (pin "1")
+    (instances
+      (project "The Luwu PCB"
+        (path "/12a97621-0282-4218-86a3-43268902dd9c"
+          (reference "H2") (unit 1)
+        )
+      )
+    )
+  )
   (symbol (lib_id "power:GND") (at 195.58 126.365 0) (unit 1)
     (in_bom yes) (on_board yes) (dnp no) (fields_autoplaced)
@@
     )
   )
+  (symbol (lib_id "power:GND") (at 47.625 149.225 0) (unit 1)
+    (in_bom yes) (on_board yes) (dnp no) (fields_autoplaced)
+    (property "Reference" "#PWR050" (at 47.625 155.575 0)
+      (effects (font (size 1.27 1.27)) hide)
+    )
+    (property "Value" "GND" (at 47.625 153.67 0)
+      (effects (font (size 1.27 1.27)))
+    )
+    (property "Footprint" "" (at 47.625 149.225 0)
+      (effects (font (size 1.27 1.27)) hide)
+    )
+    (property "Datasheet" "" (at 47.625 149.225 0)
+      (effects (font (size 1.27 1.27)) hide)
+    )
+    (pin "1")
+    (instances
+      (project "The Luwu PCB"
+        (path "/12a97621-0282-4218-86a3-43268902dd9c"
+          (reference "#PWR050") (unit 1)
+        )
+      )
+    )
+  )
+  (symbol (lib_id "power:GND") (at 70.485 149.225 0) (unit 1)
+    (in_bom yes) (on_board yes) (dnp no) (fields_autoplaced)
+    (property "Reference" "#PWR051" (at 70.485 155.575 0)
+      (effects (font (size 1.27 1.27)) hide)
+    )
+    (property "Value" "GND" (at 70.485 153.67 0)
+      (effects (font (size 1.27 1.27)))
+    )
+    (property "Footprint" "" (at 70.485 149.225 0)
+      (effects (font (size 1.27 1.27)) hide)
+    )
+    (property "Datasheet" "" (at 70.485 149.225 0)
+      (effects (font (size 1.27 1.27)) hide)
+    )
+    (pin "1")
+    (instances
+      (project "The Luwu PCB"
+        (path "/12a97621-0282-4218-86a3-43268902dd9c"
+          (reference "#PWR051") (unit 1)
+        )
+      )
+    )
+  )
   (symbol (lib_id "power:+12V") (at 163.195 44.45 0) (unit 1)
     (in_bom yes) (on_board yes) (dnp no) (fields_autoplaced)
@@
         )
       )
+    )
+  )
+  (symbol (lib_id "power:GND") (at 24.765 149.225 0) (unit 1)
+    (in_bom yes) (on_board yes) (dnp no) (fields_autoplaced)
+    (property "Reference" "#PWR049" (at 24.765 155.575 0)
+      (effects (font (size 1.27 1.27)) hide)
+    )
+    (property "Value" "GND" (at 24.765 153.67 0)
+      (effects (font (size 1.27 1.27)))
+    )
+    (property "Footprint" "" (at 24.765 149.225 0)
+      (effects (font (size 1.27 1.27)) hide)
+    )
+    (property "Datasheet" "" (at 24.765 149.225 0)
+      (effects (font (size 1.27 1.27)) hide)
+    )
+    (pin "1")
+    (instances
+      (project "The Luwu PCB"
+        (path "/12a97621-0282-4218-86a3-43268902dd9c"
+          (reference "#PWR049") (unit 1)
+        )
+      )

Commit message: updated size
Parts:
- removed J10: Neopixel Terminal out 3, TerminalBlock:TerminalBlock_bornier-3_P5.08mm, symbol Connector:Screw_Terminal_01x03
- removed J3: 5V_IN, TerminalBlock:TerminalBlock_bornier-2_P5.08mm, symbol Connector:Screw_Terminal_01x02
- removed J4: Neopixel Terminal opt 1, TerminalBlock:TerminalBlock_bornier-3_P5.08mm, symbol Connector:Screw_Terminal_01x03
- removed J5: 12V_IN, TerminalBlock:TerminalBlock_bornier-2_P5.08mm, symbol Connector:Screw_Terminal_01x02
- removed J7: Screw_Terminal_01x04, TerminalBlock:TerminalBlock_bornier-4_P5.08mm, symbol Connector:Screw_Terminal_01x04
- removed J8: Neopixel Terminal, TerminalBlock:TerminalBlock_bornier-3_P5.08mm, symbol Connector:Screw_Terminal_01x03
- removed J9: Neopixel Terminal opt 2, TerminalBlock:TerminalBlock_bornier-3_P5.08mm, symbol Connector:Screw_Terminal_01x03
- added J11: Screw_Terminal_01x14, Connector_custom:TerminalBlock_bornier-14_P5.08mm, symbol Connector:Screw_Terminal_01x14
- added J4: Screw_Terminal_01x06, TerminalBlock:TerminalBlock_bornier-6_P5.08mm, symbol Connector:Screw_Terminal_01x06
Connections:
- net +12V: now also J11.2 (Pin_2), J11.3 (Pin_3)
- net +5V: now also J11.12 (Pin_12), J11.9 (Pin_9), J4.1 (Pin_1), J4.4 (Pin_4)
- net 5V_IN_TERM: now also J11.8 (Pin_8)
- net DATA 1 OUT: now also J4.5 (Pin_5)
- net DATA OPT1 OUT: now also J11.13 (Pin_13)
- net DATA OPT2 OUT: now also J11.10 (Pin_10)
- net DATA OPT3 OUT: now also J4.2 (Pin_2)
- net GND: now also J11.1 (Pin_1), J11.11 (Pin_11), J11.14 (Pin_14), J11.7 (Pin_7), J4.3 (Pin_3), J4.6 (Pin_6)
- net LED_B: now also J11.6 (Pin_6)
- net LED_G: now also J11.5 (Pin_5)
- net LED_R: now also J11.4 (Pin_4)
